File: VIPR_PCB/PiHAT_SSR_V4/PiHAT_SSR_V4.brd (EAGLE design)
At the start: 65 x 68.7 mm, 35 parts, among them CN1 M12_8PIN_CODE_A

Commit message: Add files via upload
Parts:
- AUML1: device MyLibrary:SMD-SPECIAL_28PIN_PIC32_11_3_2011_MOD5_20_13_SMT_CAP_2220 -> VIPR_Components:SMD-SPECIAL_28PIN_PIC32_11_3_2011_MOD5_20_13_SMT_CAP_2220
- CN1: device MyLibrary:M12_8PIN_CODE_A -> VIPR_Components:M12_8PIN_CODE_A
- D1: device MyLibrary:SCHOTTKY_DIODE_SMD_DO-214AB -> VIPR_Components:SCHOTTKY_DIODE_SMD_DO-214AB
- J1, J2, J3, J4, J5: device MyLibrary:1X01 -> VIPR_Components:1X01
- J6, J7: device MyLibrary:1X02_BIG -> VIPR_Components:1X02_BIG
- JP1: device MyLibrary:2X20 -> VIPR_Components:2X20
- SSR1, SSR2, SSR3, SSR4: device MyLibrary:OMRON_G3VM-101FR -> VIPR_Components:OMRON_G3VM-101FR
- VR1, VR2: device MyLibrary:SMD-SPECIAL_28PIN_PIC32_11_3_2011_DPAK-5 -> VIPR_Components:SMD-SPECIAL_28PIN_PIC32_11_3_2011_DPAK-5

Commit message: Add files via upload
Parts:
- added D2, D3, D4: SCHOTTKY_DIODE_SS310L_DO_219AB, VIPR_Components:SCHOTTKY_DIODE_DO219AB
- added J10: GPIO_5 (OUT), VIPR_Components:1X01
- added J11: GPIO_17 (IN), VIPR_Components:1X01
- added J12: GPIO_12, VIPR_Components:1X01
- added J13: (no value), VIPR_Components:1X02_BIG
- added J8: GPIO_13 (OUT), VIPR_Components:1X01
- added J9: GPIO_6 (OUT), VIPR_Components:1X01
- added R1: 665, rcl:M0805
- added R10: (no value), rcl:R2512
- added R5: 170k, rcl:M0805
- R6: value 170k -> 100k
- R7: value 100k -> 1.2k
- R8: value 1.2k -> (none); device rcl:M0805 -> rcl:R2512
- R9: value 665 -> (none); device rcl:M0805 -> rcl:R2512
- moved R6 44.1 mm to (3.40, 37.2), turned to 270 degrees
- moved R9 36.4 mm to (41.0, 42.0), turned to 270 degrees
- moved R8 34.4 mm to (54.0, 42.0), turned to 270 degrees
- moved R4 27.2 mm to (8.30, 58.1), turned to 90 degrees
- moved R7 18.0 mm to (19.7, 44.9), turned to 180 degrees
- moved SSR1 13.0 mm to (58.0, 52.0)
- moved SSR2 13.0 mm to (45.0, 52.0)
- moved R2 12.1 mm to (47.0, 59.3), turned to 180 degrees
- moved R3 11.5 mm to (35.5, 59.2)
Connections:
- removed net N$4 (its old number): R3.2, SSR1.P$2
- new net N$1: D2.P$2, R8.2
- new net N$3: D3.P$2, R9.2
- new net N$5: R1.2, SSR1.P$2
- new net N$7: D4.P$2, R10.2
- net 3V3: now also R4.2; no longer R9.2
- net ENABLE_SOL_12V: now also R7.1; no longer R8.1
- net GND: now also R5.1; no longer R7.1
- net GPIO_12: now also J12.1; no longer R3.1
- net GPIO_13: now also J8.1, R1.1; no longer R2.1
- net GPIO_17: now also J11.1, R4.1; no longer R9.1
- net GPIO_5: now also J10.1, R3.1
- net GPIO_6: now also J9.1, R2.1; no longer R4.1
- net N$2: now also R3.2; no longer R4.2
- net N$6: now also R7.2; no longer R8.2
- net SOL_1: now also CN1.P$5, R10.1, SSR3.P$6, SSR3.P$7; no longer CN1.P$4, SSR1.P$6, SSR1.P$7
- net SOL_12V: now also J13.P$1
- net SOL_2: now also R8.1, SSR1.P$6, SSR1.P$7; no longer SSR2.P$6, SSR2.P$7
- net SOL_3: now also CN1.P$4, R9.1, SSR2.P$6, SSR2.P$7; no longer CN1.P$5, SSR3.P$6, SSR3.P$7
- net SOL_GND: now also D2.P$1, D3.P$1, D4.P$1, J13.P$2
- net VSET_5V: now also R6.2; no longer R7.2
- net VSET_8V5: now also R5.2; no longer R6.2
Routing:
- net GPIO_12: track 7.50 -> 27.4 mm
- net GPIO_5: track 0.00 -> 17.8 mm
- net SOL_1: track 45.4 -> 59.6 mm
- net GND: track 36.9 -> 45.0 mm, vias 10 -> 13
- net SOL_GND: track 2.39 -> 8.30 mm, vias 1 -> 4
- net GPIO_13: track 12.3 -> 18.0 mm
- net N$7: track 0.00 -> 4.53 mm
- net N$3: track 0.00 -> 4.53 mm
- net N$1: track 0.00 -> 4.53 mm
- net SOL_2: track 47.3 -> 51.4 mm
- net GPIO_17: track 22.3 -> 25.5 mm
- net N$4 (its old number): track 3.12 -> 0.00 mm
- net ENABLE_SOL_12V: track 58.8 -> 55.9 mm
- net SOL_3: track 52.4 -> 49.7 mm
- net N$5: track 0.00 -> 2.65 mm
Other:
- board text added: "+"
- board text added: "PiHAT_SSRelay_V4_3_23_2020"
- board text added: "Solenoid 12V"
- board text removed: "PiHAT_SSRelay_V3_2_28_2019"
