File: VIPR_PCB/PiHAT_SSR_V4/PiHAT_SSR_V4.sch (EAGLE design)
At the start: 35 parts, among them CN1 M12_8PIN_CODE_A

Commit message: Add files via upload
Parts:
- AUML1: device MyLibrary:SMD-SPECIAL_28PIN_PIC32_11_3_2011_MOD5_20_13_AUML_MULTI-LAYER-VARISTOR -> VIPR_Components:SMD-SPECIAL_28PIN_PIC32_11_3_2011_MOD5_20_13_AUML_MULTI-LAYER-VARISTOR
- CN1: device MyLibrary:M12_8PIN_CODE_A -> VIPR_Components:M12_8PIN_CODE_A
- D1: device MyLibrary:SCHOTTKY_DIODE_4A -> VIPR_Components:SCHOTTKY_DIODE_4A
- J1, J2, J3, J4, J5: device MyLibrary:CONN_01 -> VIPR_Components:CONN_01
- J6, J7: device MyLibrary:CONN_02PTH2 -> VIPR_Components:CONN_02PTH2
- JP1: device MyLibrary:40W_PI_HAT_TPH -> VIPR_Components:40W_PI_HAT_TPH
- SSR1, SSR2, SSR3, SSR4: device MyLibrary:OMRON_G3VM_101FR -> VIPR_Components:OMRON_G3VM_101FR
- VR1, VR2: device MyLibrary:SMD-SPECIAL_28PIN_PIC32_11_3_2011_LT3083 -> VIPR_Components:SMD-SPECIAL_28PIN_PIC32_11_3_2011_LT3083
Changed lines of the file:
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@@
 </classes>
 <parts>
-<part name="JP1" library="MyLibrary" deviceset="40W_PI_HAT_TPH" device=""/>
+<part name="JP1" library="VIPR_Components" deviceset="40W_PI_HAT_TPH" device=""/>
 <part name="R3" library="rcl" library_urn="urn:adsk.eagle:library:334" deviceset="R-US_" device="M0805" package3d_urn="urn:adsk.eagle:package:23556/2" value="665"/>
 <part name="R2" library="rcl" library_urn="urn:adsk.eagle:library:334" deviceset="R-US_" device="M0805" package3d_urn="urn:adsk.eagle:package:23556/2" value="665"/>
 <part name="R4" library="rcl" library_urn="urn:adsk.eagle:library:334" deviceset="R-US_" device="M0805" package3d_urn="urn:adsk.eagle:package:23556/2" value="665"/>
-<part name="VR1" library="MyLibrary" deviceset="SMD-SPECIAL_28PIN_PIC32_11_3_2011_LT3083" device=""/>
+<part name="VR1" library="VIPR_Components" deviceset="SMD-SPECIAL_28PIN_PIC32_11_3_2011_LT3083" device=""/>
 <part name="C1" library="rcl" library_urn="urn:adsk.eagle:library:334" deviceset="C-EU" device="C0805" package3d_urn="urn:adsk.eagle:package:23617/2" value="0.1uF"/>
 <part name="R6" library="rcl" library_urn="urn:adsk.eagle:library:334" deviceset="R-US_" device="M0805" package3d_urn="urn:adsk.eagle:package:23556/2" value="170k"/>
@@
 <part name="C4" library="rcl" library_urn="urn:adsk.eagle:library:334" deviceset="C-EU" device="C0805" package3d_urn="urn:adsk.eagle:package:23617/2" value="0.01uF"/>
 <part name="C5" library="rcl" library_urn="urn:adsk.eagle:library:334" deviceset="C-EU" device="C0805" package3d_urn="urn:adsk.eagle:package:23617/2" value="10uF"/>
-<part name="CN1" library="MyLibrary" deviceset="M12_8PIN_CODE_A" device=""/>
-<part name="AUML1" library="MyLibrary" deviceset="SMD-SPECIAL_28PIN_PIC32_11_3_2011_MOD5_20_13_AUML_MULTI-LAYER-VARISTOR" device=""/>
+<part name="CN1" library="VIPR_Components" deviceset="M12_8PIN_CODE_A" device=""/>
+<part name="AUML1" library="VIPR_Components" deviceset="SMD-SPECIAL_28PIN_PIC32_11_3_2011_MOD5_20_13_AUML_MULTI-LAYER-VARISTOR" device=""/>
 <part name="C6" library="rcl" library_urn="urn:adsk.eagle:library:334" deviceset="C-EU" device="C2220K" package3d_urn="urn:adsk.eagle:package:23687/2" value="10uF, 100V"/>
-<part name="D1" library="MyLibrary" deviceset="SCHOTTKY_DIODE_4A" device=""/>
+<part name="D1" library="VIPR_Components" deviceset="SCHOTTKY_DIODE_4A" device=""/>
 <part name="R8" library="rcl" library_urn="urn:adsk.eagle:library:334" deviceset="R-US_" device="M0805" package3d_urn="urn:adsk.eagle:package:23556/2" value="1.2k"/>
 <part name="R9" library="rcl" library_urn="urn:adsk.eagle:library:334" deviceset="R-US_" device="M0805" package3d_urn="urn:adsk.eagle:package:23556/2" value="665"/>
-<part name="VR2" library="MyLibrary" deviceset="SMD-SPECIAL_28PIN_PIC32_11_3_2011_LT3083" device=""/>
+<part name="VR2" library="VIPR_Components" deviceset="SMD-SPECIAL_28PIN_PIC32_11_3_2011_LT3083" device=""/>
 <part name="C7" library="rcl" library_urn="urn:adsk.eagle:library:334" deviceset="C-EU" device="C0805" package3d_urn="urn:adsk.eagle:package:23617/2" value="0.1uF"/>
 <part name="R7" library="rcl" library_urn="urn:adsk.eagle:library:334" deviceset="R-US_" device="M0805" package3d_urn="urn:adsk.eagle:package:23556/2" value="100k"/>
@@
 <part name="C10" library="rcl" library_urn="urn:adsk.eagle:library:334" deviceset="C-EU" device="C0805" package3d_urn="urn:adsk.eagle:package:23617/2" value="10uF"/>
 <part name="C11" library="rcl" library_urn="urn:adsk.eagle:library:334" deviceset="C-EU" device="C0805" package3d_urn="urn:adsk.eagle:package:23617/2" value="0.1uF"/>
-<part name="J2" library="MyLibrary" deviceset="CONN_01" device=""/>
-<part name="J3" library="MyLibrary" deviceset="CONN_01" device=""/>
-<part name="J4" library="MyLibrary" deviceset="CONN_01" device=""/>
-<part name="J5" library="MyLibrary" deviceset="CONN_01" device=""/>
-<part name="J7" library="MyLibrary" deviceset="CONN_02" device="PTH2"/>
-<part name="J6" library="MyLibrary" deviceset="CONN_02" device="PTH2"/>
-<part name="J1" library="MyLibrary" deviceset="CONN_01" device=""/>
-<part name="SSR2" library="MyLibrary" deviceset="OMRON_G3VM_101FR" device=""/>
-<part name="SSR1" library="MyLibrary" deviceset="OMRON_G3VM_101FR" device=""/>
-<part name="SSR3" library="MyLibrary" deviceset="OMRON_G3VM_101FR" device=""/>
-<part name="SSR4" library="MyLibrary" deviceset="OMRON_G3VM_101FR" device=""/>
+<part name="J2" library="VIPR_Components" deviceset="CONN_01" device=""/>
+<part name="J3" library="VIPR_Components" deviceset="CONN_01" device=""/>
+<part name="J4" library="VIPR_Components" deviceset="CONN_01" device=""/>
+<part name="J5" library="VIPR_Components" deviceset="CONN_01" device=""/>
+<part name="J7" library="VIPR_Components" deviceset="CONN_02" device="PTH2"/>
+<part name="J6" library="VIPR_Components" deviceset="CONN_02" device="PTH2"/>
+<part name="J1" library="VIPR_Components" deviceset="CONN_01" device=""/>
+<part name="SSR2" library="VIPR_Components" deviceset="OMRON_G3VM_101FR" device=""/>
+<part name="SSR1" library="VIPR_Components" deviceset="OMRON_G3VM_101FR" device=""/>
+<part name="SSR3" library="VIPR_Components" deviceset="OMRON_G3VM_101FR" device=""/>
+<part name="SSR4" library="VIPR_Components" deviceset="OMRON_G3VM_101FR" device=""/>
 </parts>
 <sheets>

Commit message: Add files via upload
Parts:
- added D2, D3, D4: SCHOTTKY_DIODE_SS310L_DO_219AB, VIPR_Components:SCHOTTKY_DIODE_SS310L_DO_219AB
- added J10: GPIO_5 (OUT), VIPR_Components:CONN_01
- added J11: GPIO_17 (IN), VIPR_Components:CONN_01
- added J12: GPIO_12, VIPR_Components:CONN_01
- added J13: (no value), VIPR_Components:CONN_02PTH2
- added J8: GPIO_13 (OUT), VIPR_Components:CONN_01
- added J9: GPIO_6 (OUT), VIPR_Components:CONN_01
- added R1: 665, rcl:R-US_M0805
- added R10: (no value), rcl:R-US_R2512
- added R5: 170k, rcl:R-US_M0805
- R6: value 170k -> 100k
- R7: value 100k -> 1.2k
- R8: value 1.2k -> (none); device rcl:R-US_M0805 -> rcl:R-US_R2512
- R9: value 665 -> (none); device rcl:R-US_M0805 -> rcl:R-US_R2512
Connections:
- removed net N$4 (its old number): R3.2, SSR1.A(2)
- new net N$1: D2.C, R8.2
- new net N$3: D3.C, R9.2
- new net N$5: R1.2, SSR1.A(2)
- new net N$7: D4.C, R10.2
- net 3V3: now also R4.2; no longer R9.2
- net ENABLE_SOL_12V: now also R7.1; no longer R8.1
- net GND: now also R5.1; no longer R7.1
- net GPIO_12: now also J12.1; no longer R3.1
- net GPIO_13: now also J8.1, R1.1; no longer R2.1
- net GPIO_17: now also J11.1, R4.1; no longer R9.1
- net GPIO_5: now also J10.1, R3.1
- net GPIO_6: now also J9.1, R2.1; no longer R4.1
- net N$2: now also R3.2; no longer R4.2
- net N$6: now also R7.2; no longer R8.2
- net SOL_1: now also CN1.P$5, R10.1, SSR3.GND(6), SSR3.GND(7); no longer CN1.P$4, SSR1.GND(6), SSR1.GND(7)
- net SOL_12V: now also J13.1
- net SOL_2: now also R8.1, SSR1.GND(6), SSR1.GND(7); no longer SSR2.GND(6), SSR2.GND(7)
- net SOL_3: now also CN1.P$4, R9.1, SSR2.GND(6), SSR2.GND(7); no longer CN1.P$5, SSR3.GND(6), SSR3.GND(7)
- net SOL_GND: now also D2.A, D3.A, D4.A, J13.2
- net VSET_5V: now also R6.2; no longer R7.2
- net VSET_8V5: now also R5.2; no longer R6.2
Other:
- note added: "SSRelay 1 - Middle/main switched solenoid/air-knife"
- note added: "SSRelay 2 - Neighboring right-side switched solenoid/air-knife"
- note added: "SSRelay 3 - Neighboring left-side switched solenoid/air-knife"
- note removed: "SSRelay 1 - Neighboring left-side switched solenoid/air-knife"
- note removed: "SSRelay 2 - Middle/main switched solenoid/air-knife"
- note removed: "SSRelay 3 - Neighboring right-side switched solenoid/air-knife"
- moved on the sheet: R2, R3, R4, R6, R8, R9
